File: realop1_burnwire_top2/realop1_burnwire_top2.kicad_pcb (KiCad board)
At the start: 2 copper layers, 98 x 98 mm, 31 parts, among them J1 BURNWIRE_SUPPLY, J2 pyro0, J3 pyro1, J4 photodiode, Q1 BSC0702LS, Q2 BSC0702LS, U1 LMV321, U2 LMV321

Commit message: Add files via upload
Parts:
- removed R1, R10, R2, R8: NiCr, RPRP_neo:nichrome_m3_pos40
- added Bottom1: MountingHole_3.2mm_M3_ISO7380_Pad_TopBottom, MountingHole:MountingHole_3.2mm_M3_ISO7380_Pad_TopBottom, F.Cu at (133.0, 137.8)
- added Bottom2: MountingHole_3.2mm_M3_ISO7380_Pad_TopBottom, MountingHole:MountingHole_3.2mm_M3_ISO7380_Pad_TopBottom, F.Cu at (156.1, 137.9)
- added Left1: MountingHole_3.2mm_M3_ISO7380_Pad_TopBottom, MountingHole:MountingHole_3.2mm_M3_ISO7380_Pad_TopBottom, F.Cu at (103.6, 85.4)
- added Left2: MountingHole_3.2mm_M3_ISO7380_Pad_TopBottom, MountingHole:MountingHole_3.2mm_M3_ISO7380_Pad_TopBottom, F.Cu at (103.6, 108.6)
- added REF**: PinHeader_1x02_P2.54mm_Vertical, Connector_PinHeader_2.54mm:PinHeader_1x02_P2.54mm_Vertical, F.Cu at (97.8, 102.8)
- added REF**: PinHeader_1x02_P2.54mm_Vertical, Connector_PinHeader_2.54mm:PinHeader_1x02_P2.54mm_Vertical, F.Cu at (188.8, 91.2)
- added REF**: PinHeader_1x02_P2.54mm_Vertical, Connector_PinHeader_2.54mm:PinHeader_1x02_P2.54mm_Vertical, F.Cu at (150.3, 143.7)
- added REF**: PinHeader_1x02_P2.54mm_Vertical, Connector_PinHeader_2.54mm:PinHeader_1x02_P2.54mm_Vertical, F.Cu at (97.8, 91.2)
- added REF**: PinHeader_1x02_P2.54mm_Vertical, Connector_PinHeader_2.54mm:PinHeader_1x02_P2.54mm_Vertical, F.Cu at (138.8, 50.2)
- added REF**: PinHeader_1x02_P2.54mm_Vertical, Connector_PinHeader_2.54mm:PinHeader_1x02_P2.54mm_Vertical, F.Cu at (188.6, 102.8)
- added REF**: PinHeader_1x02_P2.54mm_Vertical, Connector_PinHeader_2.54mm:PinHeader_1x02_P2.54mm_Vertical, F.Cu at (150.3, 50.3)
- added REF**: PinHeader_1x02_P2.54mm_Vertical, Connector_PinHeader_2.54mm:PinHeader_1x02_P2.54mm_Vertical, F.Cu at (138.7, 143.8)
- added Right1: MountingHole_3.2mm_M3_ISO7380_Pad_TopBottom, MountingHole:MountingHole_3.2mm_M3_ISO7380_Pad_TopBottom, F.Cu at (185.4, 85.5)
- added Right2: MountingHole_3.2mm_M3_ISO7380_Pad_TopBottom, MountingHole:MountingHole_3.2mm_M3_ISO7380_Pad_TopBottom, F.Cu at (185.5, 108.6)
- added Top1: MountingHole_3.2mm_M3_ISO7380_Pad_TopBottom, MountingHole:MountingHole_3.2mm_M3_ISO7380_Pad_TopBottom, F.Cu at (132.9, 56.0)
- added Top2: MountingHole_3.2mm_M3_ISO7380_Pad_TopBottom, MountingHole:MountingHole_3.2mm_M3_ISO7380_Pad_TopBottom, F.Cu at (156.1, 56.0)
- moved D3 24.3 mm to (156.2, 85.4), turned to -135 degrees
- moved R18 18.5 mm to (160.6, 83.0), turned to 135 degrees
- moved U1 14.1 mm to (162.4, 81.3), turned to -45 degrees
- moved R16 13.9 mm to (162.4, 85.3), turned to 45 degrees
- moved C3 13.3 mm to (171.4, 90.9), turned to 180 degrees
- moved R7 12.5 mm to (174.8, 92.7)
- moved R17 12.1 mm to (164.6, 83.2), turned to -135 degrees
- moved R12 11.4 mm to (173.9, 90.4), turned to -90 degrees
- moved R9 10.7 mm to (174.8, 94.2), turned to 180 degrees
- moved R15 9.46 mm to (170.1, 78.6), turned to 135 degrees
- moved R14 9.20 mm to (167.9, 79.8), turned to 45 degrees
- moved Q2 8.66 mm to (178.3, 89.2)
- moved U2 7.33 mm to (166.8, 77.2), turned to -135 degrees
- moved C2 6.91 mm to (164.4, 79.4), turned to 135 degrees
- moved R3 6.12 mm to (164.8, 75.4), turned to 45 degrees
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Routing:
- net /3v3_tia: track 0.00 -> 25.8 mm, vias 6 -> 0
- net /pd_tia0: track 41.1 -> 20.0 mm
- net Net-(Q2-G): track 10.5 -> 0.00 mm
- net /pyro1_cs: track 36.2 -> 30.5 mm
- net Net-(D3-K): track 5.50 -> 0.00 mm
- net /pd_tia1: track 32.9 -> 27.4 mm
- net Net-(D1-K): track 5.17 -> 0.00 mm
- net Net-(U2-+): track 3.39 -> 0.00 mm
- net Net-(Q1-G): track 3.21 -> 0.00 mm
- net Net-(U1-+): track 3.38 -> 6.03 mm
- net /pyro1_enable: track 35.1 -> 32.5 mm
- net GND: vias 112 -> 133
- added copper zone on F.Cu, net (none)
- added copper zone on F.Cu, net Net-(D1-K)
- added copper zone on F.Cu, net Net-(D3-K)
- added copper zone on F.Cu, net Net-(Q1-G)
- added copper zone on F.Cu, net Net-(Q2-G)
- added copper zone on F.Cu, net Net-(U2-+)
- removed copper zone on B.Cu, net /3v3_tia
