File: realop1_powerdis_bak1/realop1_powerdis_bak1.kicad_pcb (KiCad board)
At the start: 4 copper layers, 90 x 90 mm, 97 parts, among them J1 mnt_fltctrl, J10 bsw3, J11 ground_charge, J12 picoblade_1x4, J13 mgmt_if, J14 xt30_2x, J15 picoblade_1x4, J16 picoblade_1x4, J17 test_DNP, J18 Conn_01x04, J2 picoblade_1x4, J3 Conn_01x08_MountingPin, J4 picoblade_1x4, J5 picoblade_1x4, J6 picoblade_1x4, J7 picoblade_1x4, J8 bsw1, J9 bsw2, Q1 2N7002E, Q10 MMBT3906, Q2 2N7002E, Q3 SQJ479EP, Q4 SQJ479EP, Q5 2N7002E, Q6 SQJ479EP, Q7 2N7002E, Q8 SQJ479EP, Q9 MMBT3906, U1 AP64350 / AP64352Q, U2 INA3221, U3 LP5907MFX-3.3, U4 INA3221, U5 LGS5524, U6 TMP1075DGK, U7 TMP1075DGK

Commit message: Add files via upload
Parts:
- C11, C12, C13, C28, C7, C8, C9: value 100nF -> 1uF
- moved J14 17.4 mm to (78.1, 113.1)
- moved J2 16.9 mm to (73.2, 98.0)
- moved J15 16.8 mm to (73.2, 106.0)
- moved Q3 16.4 mm to (81.7, 95.9), turned to 90 degrees
- moved R3 16.3 mm to (87.6, 103.3)
- moved Q6 16.1 mm to (82.6, 104.2)
- moved R7 15.7 mm to (76.9, 104.1), turned to -90 degrees
- moved R5 15.0 mm to (76.9, 97.0), turned to -90 degrees
- moved Q5 13.5 mm to (89.0, 105.8), turned to 90 degrees
- moved Q2 12.3 mm to (86.5, 98.1)
- moved R2 10.4 mm to (89.0, 108.6), turned to 180 degrees
- moved R19 10.2 mm to (86.1, 100.6), turned to 0 degrees
- moved R18 10.0 mm to (83.0, 100.6), turned to 0 degrees
- moved J17 3.34 mm to (85.9, 119.6), turned to 0 degrees
Connections:
- J12 pad 2: /SCS_1- -> GND
- J12 pad 3: GND -> /SCS_1-
- J16 pad 2: /SCS_3- -> GND
- J16 pad 3: GND -> /SCS_3-
- J3 pad 1: Net-(J3-Pin_1) -> Net-(J11-Pin_1)
- J3 pad 2: Net-(J3-Pin_1) -> Net-(J3-Pin_2)
- J3 pad 3: Net-(J3-Pin_1) -> Net-(J11-Pin_1)
- J3 pad 4: Net-(J3-Pin_1) -> Net-(J3-Pin_2)
- J3 pad 6: Net-(J11-Pin_1) -> Net-(J3-Pin_2)
- J3 pad 8: Net-(J11-Pin_1) -> Net-(J3-Pin_2)
- J8 pad 1: Net-(J3-Pin_1) -> Net-(J3-Pin_2)
- J8 pad 2: Net-(J3-Pin_1) -> Net-(J3-Pin_2)
- U2 pad 10: unconnected-(U2-PV-Pad10) -> GND
- U2 pad 13: unconnected-(U2-TC-Pad13) -> GND
- U2 pad 8: unconnected-(U2-WARNING-Pad8) -> GND
- U2 pad 9: unconnected-(U2-CRITICAL-Pad9) -> GND
- U4 pad 10: unconnected-(U4-PV-Pad10) -> GND
- U4 pad 13: unconnected-(U4-TC-Pad13) -> GND
- U4 pad 8: unconnected-(U4-WARNING-Pad8) -> GND
- U4 pad 9: unconnected-(U4-CRITICAL-Pad9) -> GND
- U6 pad 3: unconnected-(U6-ALERT-Pad3) -> GND
- U7 pad 3: unconnected-(U7-ALERT-Pad3) -> GND
Routing:
- net /SCS_0+: track 14.1 -> 47.5 mm
- net /SCS_2+: track 18.2 -> 43.2 mm
- net /SCS_0-: track 24.1 -> 43.6 mm
- net /SCS_2-: track 25.2 -> 40.7 mm
- net /pwr0_en: track 81.1 -> 95.5 mm
- net /pwr2_en: track 72.8 -> 84.0 mm
- net BATPACK_V+: track 29.8 -> 31.5 mm, vias 36 -> 28
- net Net-(Q5-D): track 3.93 -> 4.95 mm
- net GND: vias 241 -> 229
- added copper zone on F.Cu, net Net-(J3-Pin_2)
- removed copper zone on B.Cu, net Net-(J3-Pin_1)
Other:
- board text added: "-+-+"
- board text added: "ABF PIN"
- board text added: "HARD-SW"
- board text added: "rop1_pdis_bak2"
- board text removed: "ANT"
- board text removed: "APPLY-BEFORE-FLIGHT"
- board text removed: "rop1_pdis_bak1"
